Commit message: Change PSM model source from dvrk_ros to dvrk_env.

File: cosur/dvrk.urdf (robot description, URDF)
Before this commit: robot dvrk_psm, 12 links, 11 joints
Links:
- removed link outer_insertion_link
- removed link outer_pitch_back_link
- removed link outer_pitch_bottom_link
- removed link outer_pitch_front_link
- removed link outer_pitch_link
- removed link outer_pitch_top_link
- removed link outer_yaw_link
- removed link psm_base_link
- removed link tool_main_link
- removed link tool_wrist_link
- removed link tool_wrist_shaft_link
- added link base_link, mass 2.0161; collision mesh filename=meshes/psm/base_link.stl; visual mesh filename=meshes/psm/base_link.stl
- added link main_insertion_link, mass 0.22491; collision mesh filename=meshes/psm/main_insertion_link.stl; visual mesh filename=meshes/psm/main_insertion_link.stl
- added link pitch_back_link, mass 0.98494; collision mesh filename=meshes/psm/pitch_back_link.stl; visual mesh filename=meshes/psm/pitch_back_link.stl
- added link pitch_bottom_link, mass 0.44569; collision mesh filename=meshes/psm/pitch_bottom_link.stl; visual mesh filename=meshes/psm/pitch_bottom_link.stl
- added link pitch_end_link, mass 2.091; collision mesh filename=meshes/psm/pitch_end_link.stl; visual mesh filename=meshes/psm/pitch_end_link.stl
- added link pitch_front_link, mass 0.074425; collision mesh filename=meshes/psm/pitch_front_link.stl; visual mesh filename=meshes/psm/pitch_front_link.stl
- added link pitch_top_link, mass 0.17841; collision mesh filename=meshes/psm/pitch_top_link.stl; visual mesh filename=meshes/psm/pitch_top_link.stl
- added link remote_center_link
- added link tool_gripper1_link, mass 0; collision mesh filename=meshes/psm/tool_gripper1_link.stl; visual mesh filename=meshes/psm/tool_gripper1_link.stl
- added link tool_gripper2_link, mass 0; collision mesh filename=meshes/psm/tool_gripper2_link.stl; visual mesh filename=meshes/psm/tool_gripper2_link.stl
- added link tool_pitch_link, mass 0.00025784; collision mesh filename=meshes/psm/tool_pitch_link.stl; visual mesh filename=meshes/psm/tool_pitch_link.stl
- added link tool_roll_link, mass 0.00033225; collision mesh filename=meshes/psm/tool_roll_link.stl; visual mesh filename=meshes/psm/tool_roll_link.stl
- added link tool_yaw_link, mass 0; collision mesh filename=meshes/psm/tool_yaw_link.stl; visual mesh filename=meshes/psm/tool_yaw_link.stl
- added link yaw_link, mass 1.4705; collision mesh filename=meshes/psm/yaw_link.stl; visual mesh filename=meshes/psm/yaw_link.stl
Joints:
- removed joint fixed
- removed joint outer_insertion
- removed joint outer_pitch
- removed joint outer_pitch_1
- removed joint outer_pitch_2
- removed joint outer_pitch_3
- removed joint outer_pitch_4
- removed joint outer_pitch_5
- removed joint outer_roll
- removed joint outer_roll_shaft
- removed joint outer_yaw
- added joint main_insertion_joint: type prismatic, parent pitch_end_link, child main_insertion_link, origin xyz=0.043 -0.28809 0 rpy=1.5708 1.5708 3.1416, axis 0 0 1, limit lower=0 upper=0.24 effort=1000 velocity=1
- added joint pitch_back_joint: type revolute, parent yaw_link, child pitch_back_link, origin xyz=0 0 0.0296 rpy=-1.5708 -0.29073 0, axis 0 0 1, limit lower=-0.93556 upper=0.94249 effort=1000 velocity=10
- added joint pitch_bottom_joint: type revolute, parent pitch_back_link, child pitch_bottom_link, origin xyz=0.15 0 0 rpy=0 0 1.8615, axis 0 0 1, limit lower=-0.94249 upper=0.93556 effort=1000 velocity=10, mimic joint=pitch_back_joint multiplier=-1
- added joint pitch_end_joint: type revolute, parent pitch_bottom_link, child pitch_end_link, origin xyz=0.516 0 0 rpy=0 0 0, axis 0 0 1, limit lower=-0.93556 upper=0.94249 effort=1000 velocity=10, mimic joint=pitch_back_joint multiplier=1
- added joint pitch_front_joint: type revolute, parent yaw_link, child pitch_front_link, origin xyz=0 0 -0.0664 rpy=-1.5708 -0.29073 0, axis 0 0 1, limit lower=-0.93556 upper=0.94249 effort=1000 velocity=10, mimic joint=pitch_back_joint multiplier=1
- added joint pitch_top_joint: type revolute, parent pitch_back_link, child pitch_top_link, origin xyz=0.18366 0.014121 0 rpy=0 0 1.8615, axis 0 0 1, limit lower=-0.94249 upper=0.93556 effort=1000 velocity=10, mimic joint=pitch_back_joint multiplier=-1
- added joint remote_center_joint: type fixed, parent base_link, child remote_center_link, origin xyz=0 0.4864 0 rpy=0 0 0
- added joint rev_joint: type revolute, parent world, child base_link, origin xyz=0 0 0 rpy=0 0 0, axis 0 0 1, limit lower=-3.14159 upper=3.14159 effort=1000 velocity=10
- added joint tool_gripper1_joint: type revolute, parent tool_yaw_link, child tool_gripper1_link, origin xyz=0 0 0 rpy=0 0 0, axis 0 0 1, limit lower=0 upper=1 effort=0 velocity=0, mimic joint=tool_gripper2_joint multiplier=-1
- added joint tool_gripper2_joint: type revolute, parent tool_yaw_link, child tool_gripper2_link, origin xyz=0 0 0 rpy=0 0 0, axis 0 0 1, limit lower=0 upper=1 effort=0 velocity=0
- added joint tool_pitch_joint: type revolute, parent tool_roll_link, child tool_pitch_link, origin xyz=0 0 0 rpy=1.5708 -1.5708 3.1416, axis 0 0 1, limit lower=-1.5708 upper=1.5708 effort=1000 velocity=10
- added joint tool_roll_joint: type revolute, parent main_insertion_link, child tool_roll_link, origin xyz=0 0 0.4162 rpy=0 0 -1.5708, axis 0 0 1, limit lower=-3.14159 upper=3.14159 effort=1000 velocity=10
- added joint tool_yaw_joint: type revolute, parent tool_pitch_link, child tool_yaw_link, origin xyz=0.0091 0 0 rpy=1.5708 -1.5708 3.1416, axis 0 0 1, limit lower=-1.5708 upper=1.5708 effort=1000 velocity=10
- added joint yaw_joint: type revolute, parent base_link, child yaw_link, origin xyz=0 0 0 rpy=1.5708 -1.5708 0, axis 0 0 1, limit lower=-1.605 upper=1.5994 effort=1000 velocity=10

Commit message: Move coupled PSM joints together.

File: cosur/dvrk.urdf (robot description, URDF)
Before this commit: robot psm, 15 links, 14 joints
Joints:
- joint rev_joint: axis 0 0 1 -> (none); limit lower=-3.14159 upper=3.14159 effort=1000 velocity=10 -> (none); type revolute -> fixed

Commit message: Add temporary script to test simulating the mechanically coupled links of the PSM with pybullet's createConstraint.

File: cosur/dvrk.urdf (robot description, URDF)
Before this commit: robot psm, 15 links, 14 joints
Links:
- removed link world
Joints:
- removed joint rev_joint
- joint pitch_back_joint: type revolute -> continuous
- joint pitch_bottom_joint: type revolute -> continuous
- joint pitch_end_joint: type revolute -> continuous
- joint pitch_front_joint: type revolute -> continuous
- joint pitch_top_joint: type revolute -> continuous
- joint tool_gripper1_joint: type revolute -> continuous
- joint tool_gripper2_joint: type revolute -> continuous
- joint tool_pitch_joint: type revolute -> continuous
- joint tool_roll_joint: type revolute -> continuous
- joint tool_yaw_joint: type revolute -> continuous
- joint yaw_joint: type revolute -> continuous

Commit message: Add a fake link to the EE with a spherical joint for grasping the cloth. Increase maximum effort of joints. Add cloth with attachements to the scene. Change actuation from forcing joint values to pybullet's motor control function (PD controller). Create Gymnasium env.

File: cosur/dvrk.urdf (robot description, URDF)
Before this commit: robot psm, 14 links, 13 joints
Links:
- added link grasp_link, mass 0.003; visual sphere radius=0.003
Joints:
- added joint grasp_joint: type spherical, parent tool_yaw_link, child grasp_link, origin xyz=0 0 0 rpy=0 0 0
- joint main_insertion_joint: limit lower=0 upper=0.24 effort=1000 velocity=1 -> lower=0 upper=0.24 effort=1000000 velocity=1
- joint pitch_back_joint: limit lower=-0.93556 upper=0.94249 effort=1000 velocity=10 -> lower=-0.93556 upper=0.94249 effort=1000000 velocity=10
- joint pitch_bottom_joint: limit lower=-0.94249 upper=0.93556 effort=1000 velocity=10 -> lower=-0.94249 upper=0.93556 effort=1000000 velocity=10
- joint pitch_end_joint: limit lower=-0.93556 upper=0.94249 effort=1000 velocity=10 -> lower=-0.93556 upper=0.94249 effort=1000000 velocity=10
- joint pitch_front_joint: limit lower=-0.93556 upper=0.94249 effort=1000 velocity=10 -> lower=-0.93556 upper=0.94249 effort=1000000 velocity=10
- joint pitch_top_joint: limit lower=-0.94249 upper=0.93556 effort=1000 velocity=10 -> lower=-0.94249 upper=0.93556 effort=1000000 velocity=10
- joint tool_pitch_joint: limit lower=-1.5708 upper=1.5708 effort=1000 velocity=10 -> lower=-1.5708 upper=1.5708 effort=1000000 velocity=10
- joint tool_roll_joint: limit lower=-3.14159 upper=3.14159 effort=1000 velocity=10 -> lower=-3.14159 upper=3.14159 effort=1000000 velocity=10
- joint tool_yaw_joint: limit lower=-1.5708 upper=1.5708 effort=1000 velocity=10 -> lower=-1.5708 upper=1.5708 effort=1000000 velocity=10
- joint yaw_joint: limit lower=-1.605 upper=1.5994 effort=1000 velocity=10 -> lower=-1.605 upper=1.5994 effort=1000000 velocity=10

Commit message: Add (a higher) mass to the tool links, so that motor control actually works. Reduce effort limits on the joints back to initial values.

File: cosur/dvrk.urdf (robot description, URDF)
Before this commit: robot psm, 15 links, 14 joints
Links:
- link tool_gripper1_link: mass 0 -> 0.01
- link tool_gripper2_link: mass 0 -> 0.01
- link tool_pitch_link: mass 0.00025784 -> 0.03
- link tool_roll_link: mass 0.00033225 -> 0.03
- link tool_yaw_link: mass 0 -> 0.01
Joints:
- joint main_insertion_joint: limit lower=0 upper=0.24 effort=1000000 velocity=1 -> lower=0 upper=0.24 effort=1000 velocity=1
- joint pitch_back_joint: limit lower=-0.93556 upper=0.94249 effort=1000000 velocity=10 -> lower=-0.93556 upper=0.94249 effort=1000 velocity=10
- joint pitch_bottom_joint: limit lower=-0.94249 upper=0.93556 effort=1000000 velocity=10 -> lower=-0.94249 upper=0.93556 effort=1000 velocity=10
- joint pitch_end_joint: limit lower=-0.93556 upper=0.94249 effort=1000000 velocity=10 -> lower=-0.93556 upper=0.94249 effort=1000 velocity=10
- joint pitch_front_joint: limit lower=-0.93556 upper=0.94249 effort=1000000 velocity=10 -> lower=-0.93556 upper=0.94249 effort=1000 velocity=10
- joint pitch_top_joint: limit lower=-0.94249 upper=0.93556 effort=1000000 velocity=10 -> lower=-0.94249 upper=0.93556 effort=1000 velocity=10
- joint tool_gripper1_joint: limit lower=0 upper=1 effort=0 velocity=0 -> lower=-1 upper=0 effort=0 velocity=0; mimic joint=tool_gripper2_joint multiplier=-1 -> (none)
- joint tool_pitch_joint: limit lower=-1.5708 upper=1.5708 effort=1000000 velocity=10 -> lower=-1.5708 upper=1.5708 effort=1000 velocity=10
- joint tool_roll_joint: limit lower=-3.14159 upper=3.14159 effort=1000000 velocity=10 -> lower=-3.14159 upper=3.14159 effort=1000 velocity=10
- joint tool_yaw_joint: limit lower=-1.5708 upper=1.5708 effort=1000000 velocity=10 -> lower=-1.5708 upper=1.5708 effort=1000 velocity=10
- joint yaw_joint: limit lower=-1.605 upper=1.5994 effort=1000000 velocity=10 -> lower=-1.605 upper=1.5994 effort=1000 velocity=10

Commit message: Add axis tag to spherical grasp joint.

File: cosur/dvrk.urdf (robot description, URDF)
Before this commit: robot psm, 15 links, 14 joints
Joints:
- joint grasp_joint: axis (none) -> 1 1 1
